Commit message: feat.能够实现加装末端机构的机械臂运动

File: src/jaka_ros2/src/jaka_zu20_moveit_config/config/jaka_zu20.urdf.xacro (robot description, xacro)
@@ -4,9 +4,10 @@
     <xacro:arg name="use_gazebo" default="false"/>
     <xacro:arg name="use_rviz_sim" default="false"/>
-    <!-- Import jaka_zu20 urdf file -->
     <xacro:include filename="$(find jaka_description)/urdf/jaka_zu20.urdf" />
-    <!-- Import control_xacro -->
     <xacro:include filename="jaka_zu20.ros2_control.xacro" />
-    <!-- <xacro:jaka_zu20_ros2_control name="FakeSystem" initial_positions_file="$(arg initial_positions_file)"/> -->
+    <xacro:include filename="$(find robotiq_description)/urdf/robotiq_2f_85_macro.urdf.xacro" />
     <xacro:jaka_zu20_ros2_control name="jaka_zu20_hardware" initial_positions_file="$(arg initial_positions_file)" use_gazebo="$(arg use_gazebo)" use_rviz_sim="$(arg use_rviz_sim)" />
+    <xacro:robotiq_gripper name="RobotiqGripperHardwareInterface" prefix="" parent="Link_06" use_fake_hardware="$(arg use_rviz_sim)" sim_ignition="$(arg use_gazebo)">
+        <origin xyz="0 0 0" rpy="0 0 0" />
+    </xacro:robotiq_gripper>
 </robot>
